File: ESP12 adapter/esp12-adapter.brd (EAGLE design)
At the start: 44.1 x 39.4 mm, 10 parts

Commit message: Update
Parts:
- removed U$1: ESP12, esp-12e:ESP12
- added U$2: ESP12, esp826612q:ESP12
Connections:
- net +3V3: now also U$2.VCC; no longer U$1.VCC
- net GND: now also U$2.GND; no longer U$1.GND
- net N$1: now also U$2.RESET; no longer U$1.RESET
- net N$10: now also U$2.RX; no longer U$1.RX
- net N$11: now also U$2.GPIO4; no longer U$1.GPIO4
- net N$12: now also U$2.GPIO5; no longer U$1.GPIO5
- net N$13: now also U$2.GPIO0; no longer U$1.GPIO0
- net N$14: now also U$2.GPIO2; no longer U$1.GPIO2
- net N$15: now also U$2.GPIO15; no longer U$1.GPIO15
- net N$2: now also U$2.ADC; no longer U$1.ADC
- net N$3: now also U$2.CH_PD; no longer U$1.CH_PD
- net N$4: now also U$2.GPIO16; no longer U$1.GPIO16
- net N$5: now also U$2.GPIO14; no longer U$1.GPIO14
- net N$6: now also U$2.GPIO12; no longer U$1.GPIO12
- net N$7: now also U$2.GPIO13; no longer U$1.GPIO13
- net N$9: now also U$2.TX; no longer U$1.TX
Routing:
- net N$5: track 4.81 -> 6.51 mm
- net N$13: track 5.01 -> 6.02 mm
- net +3V3: track 47.4 -> 48.4 mm
- net N$7: track 5.24 -> 6.19 mm
- net N$6: track 5.02 -> 5.96 mm
- net N$14: track 5.22 -> 6.16 mm
- net N$15: track 5.44 -> 6.39 mm
- net N$2: track 5.48 -> 6.13 mm
- net N$1: track 31.7 -> 32.4 mm
- net N$3: track 5.26 -> 5.91 mm
- net N$4: track 5.03 -> 5.68 mm
- net N$11: track 5.46 -> 6.11 mm
- net N$10: track 5.68 -> 6.33 mm
- net N$9: track 5.90 -> 6.55 mm
- net N$12: track 5.23 -> 5.88 mm
