File: ESP12 adapter/v2_esp12-adapter.brd (EAGLE design)
At the start: 58.1 x 47 mm, 19 parts, among them U1 LF33CDT-TR, U2 ESP12Q

Commit message: Update tNames layer
Parts:
- removed X1: (no value), con-ptr500:AK300/2
- added POWER: (no value), con-ptr500:AK300/2
- moved C3 11.7 mm to (43.2, 10.2), turned to 90 degrees
- moved R1 2.54 mm to (21.6, 6.35)
- renumbered S1 to RESET, S2 to FLASH
Connections:
- net GND: now also POWER.2; no longer X1.2
- net N$1: now also POWER.1; no longer X1.1
Routing:
- net N$1: track 21.5 -> 16.5 mm
- net +3V3: track 114.1 -> 118.0 mm
- net N$18: track 6.13 -> 4.18 mm
Other:
- board text added: "+"
- board text added: "-"
- board text added: "GND"
- board text added: "RXD"
- board text added: "TXD"

Commit message: Update
Parts:
- C2: device rcl:E3,5-10 -> rcl:E2,5-6E
- moved RESET 3.81 mm to (6.35, 21.6)
- moved C2 2.84 mm to (30.5, 7.62)
- moved LED1 2.84 mm to (16.5, 7.62)
- moved C1 2.54 mm to (25.4, 7.62)
- moved C3 2.54 mm to (43.2, 7.62)
- moved R1 1.27 mm to (20.3, 6.35)
- moved R5 1.27 mm to (7.62, 34.3)
Connections:
- net N$1 renamed V+
- removed net VCC: JP1.8, U2.VCC
- net +3V3: now also JP1.8, U2.VCC
Routing:
- net +3V3: track 118.0 -> 130.8 mm
- net VCC: track 7.61 -> 0.00 mm
- net RESET: track 32.0 -> 35.8 mm
- net V+: track 16.5 -> 13.9 mm
- net N$18: track 4.18 -> 2.39 mm
- net ENABLE: track 10.8 -> 10.1 mm
Other:
- board text added: "www.robotyka.net.pl"
- board text removed: "robotyka.net.pl"
